File: k3yb.it/k3yb.it.kicad_pcb (KiCad board)
At the start: 2 copper layers, 228 parts, among them U1 Nice_Nano_V2, U2 4052, U3 4052, U4 4052

Commit message: alligned component Soldering MX version
Parts:
- removed U2, U3, U4: 4052, Package_SO:SO-16_3.9x9.9mm_P1.27mm
- added U5: CD74HC4067M, Package_SO:SOIC-24W_7.5x15.4mm_P1.27mm, F.Cu at (569.5, 66.7)
- D1: footprint ScottoKeebs_Hotswap:Hotswap_Choc_V1V2_1.00u -> ScottoKeebs_Components:Diode_SOD-123; moved to B.Cu
- D10, D100, D101, D102, D103, D104, D105, D106, D107, D108, D109, D11, D110, D111, D112, D12, D13, D14, D15, D16, D17, D18, D19, D2, D20, D21, D22, D23, D24, D25, D26, D27, D28, D29, D3, D30, D31, D32, D33, D34, D35, D36, D37, D38, D39, D4, D40, D41, D42, D43, D44, D45, D46, D47, D48, D49, D5, D50, D51, D52, D53, D54, D55, D56, D57, D58, D59, D6, D60, D61, D62, D63, D64, D65, D66, D67, D68, D69, D7, D70, D71, D72, D73, D74, D75, D76, D77, D78, D79, D8, D80, D81, D82, D83, D84, D85, D86, D87, D88, D89, D9, D90, D91, D92, D93, D94, D95, D96, D97, D98, D99: moved to B.Cu
- S1: value Keyswitch -> Esc
- S10: value Keyswitch -> F9
- S100, S28: value Keyswitch -> -
- S101, S24: value Keyswitch -> 7
- S102, S25: value Keyswitch -> 8
- S103, S26: value Keyswitch -> 9
- S104: value Keyswitch -> +
- S105, S21: value Keyswitch -> 4
- S106, S22: value Keyswitch -> 5
- S107, S23: value Keyswitch -> 6
- S108, S18: value Keyswitch -> 1
- S109, S19: value Keyswitch -> 2
- S11: value Keyswitch -> F10
- S110, S20: value Keyswitch -> 3
- S111: value Keyswitch -> PAD7
- S112: value Keyswitch -> PAD8
- S12: value Keyswitch -> F11
- S13: value Keyswitch -> F12
- S14: value Keyswitch -> Stamp
- S15: value Keyswitch -> Bloc scorr
- S16: value Keyswitch -> Pause
- S17: value Keyswitch -> tilde
- S2: value Keyswitch -> F1
- S27, S92: value Keyswitch -> 0
- S29: value Keyswitch -> =
- S3: value Keyswitch -> F2
- S30: value Keyswitch -> Backspace
- S31: value Keyswitch -> PAD1
- S32: value Keyswitch -> PAD2
- S33: value Keyswitch -> Tab
- S34: value Keyswitch -> q
- S35: value Keyswitch -> w
- S36: value Keyswitch -> e
- S37: value Keyswitch -> r
- S38: value Keyswitch -> t
- S39: value Keyswitch -> y
- S4: value Keyswitch -> F3
- S40: value Keyswitch -> u
- S41: value Keyswitch -> i
- S42: value Keyswitch -> o
- S43: value Keyswitch -> p
- S44: value Keyswitch -> {
- S45: value Keyswitch -> }
- S46: value Keyswitch -> ins
- S47, S78: value Keyswitch -> up
- S48: value Keyswitch -> pg up
- S49: value Keyswitch -> Caps lock
- S5: value Keyswitch -> F4
- S50: value Keyswitch -> a
- S51: value Keyswitch -> s
- S52: value Keyswitch -> d
- S53: value Keyswitch -> f
- S54: value Keyswitch -> g
- S55: value Keyswitch -> h
- S56: value Keyswitch -> j
- S57: value Keyswitch -> k
- S58: value Keyswitch -> l
- S59: value Keyswitch -> ;
- S6: value Keyswitch -> F5
- S60: value Keyswitch -> '
- S61, S94: value Keyswitch -> enter
- S62: value Keyswitch -> del
- S63: value Keyswitch -> end
- S64: value Keyswitch -> pg dowm
- S65: value Keyswitch -> Left Shift
- S66: value Keyswitch -> \
- S67: value Keyswitch -> z
- S68: value Keyswitch -> x
- S69: value Keyswitch -> c
- S7: value Keyswitch -> F6
- S70: value Keyswitch -> v
- S71: value Keyswitch -> b
- S72: value Keyswitch -> n
- S73: value Keyswitch -> m
- S74: value Keyswitch -> ,
- S75, S93: value Keyswitch -> .
- S76, S98: value Keyswitch -> /
- S77: value Keyswitch -> right shift
- S79: value Keyswitch -> PAD3
- S8: value Keyswitch -> F7
- S80: value Keyswitch -> PAD4
- S81: value Keyswitch -> left ctrl
- S82: value Keyswitch -> win
- S83: value Keyswitch -> left alt
- S84: value Keyswitch -> space
- S85: value Keyswitch -> right alt
- S86: value Keyswitch -> fn
- S87: value Keyswitch -> menu
- S88: value Keyswitch -> right ctrl
- S89: value Keyswitch -> left
- S9: value Keyswitch -> F8
- S90: value Keyswitch -> down
- S91: value Keyswitch -> right
- S95: value Keyswitch -> PAD5
- S96: value Keyswitch -> PAD6
- S97: value Keyswitch -> num
- S99: value Keyswitch -> *
- moved D96 370.4 mm to (552.8, 38.4), turned to 90 degrees
- moved D95 347.2 mm to (533.7, 38.4), turned to 90 degrees
- moved S81 337.3 mm to (45.6, 148.0)
- moved D79 331.8 mm to (495.6, 38.4), turned to 90 degrees
- moved D80 322.2 mm to (514.7, 38.4), turned to 90 degrees
- moved S65 315.9 mm to (47.9, 128.9)
- moved S83 310.5 mm to (93.5, 148.0)
- moved S82 301.7 mm to (69.4, 148.0)
- moved S67 298.7 mm to (86.0, 128.9)
- moved S14 293.0 mm to (333.7, 43.2)
- moved S16 288.1 mm to (371.8, 43.2)
- moved S66 284.0 mm to (67.0, 128.9)
- moved D111 283.4 mm to (476.6, 38.4), turned to 90 degrees
- moved D99 281.9 mm to (443.2, 67.0), turned to 90 degrees
- moved S69 281.7 mm to (124.1, 128.9)
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Connections:
- net GND renamed LOW
- D100 pad 1: Row 7 -> Row 6
- D101 pad 1: Row 7 -> Row 6
- D102 pad 1: Row 7 -> Row 6
- D103 pad 1: Row 7 -> Row 6
- D104 pad 1: Row 7 -> Row 6
- D105 pad 1: Row 7 -> Row 6
- D106 pad 1: Row 7 -> Row 6
- D107 pad 1: Row 7 -> Row 6
- D108 pad 1: Row 7 -> Row 6
- D109 pad 1: Row 7 -> Row 6
- D110 pad 1: Row 7 -> Row 6
- D111 pad 1: Row 7 -> Row 6
- D112 pad 1: Row 7 -> Row 6
- D15 pad 1: Row 1 -> Row 0
- D16 pad 1: Row 1 -> Row 0
- D29 pad 1: Row 2 -> Row 1
- D30 pad 1: Row 2 -> Row 1
- D31 pad 1: Row 2 -> Row 1
- D32 pad 1: Row 2 -> Row 1
- D43 pad 1: Row 3 -> Row 2
- D44 pad 1: Row 3 -> Row 2
- D45 pad 1: Row 3 -> Row 2
- D46 pad 1: Row 3 -> Row 2
- D47 pad 1: Row 3 -> Row 2
- D48 pad 1: Row 3 -> Row 2
- D57 pad 1: Row 4 -> Row 3
- D58 pad 1: Row 4 -> Row 3
- D59 pad 1: Row 4 -> Row 3
- D60 pad 1: Row 4 -> Row 3
- D61 pad 1: Row 4 -> Row 3
- D62 pad 1: Row 4 -> Row 3
- D63 pad 1: Row 4 -> Row 3
- D64 pad 1: Row 4 -> Row 3
- D71 pad 1: Row 5 -> Row 4
- D72 pad 1: Row 5 -> Row 4
- D73 pad 1: Row 5 -> Row 4
- D74 pad 1: Row 5 -> Row 4
- D75 pad 1: Row 5 -> Row 4
- D76 pad 1: Row 5 -> Row 4
- D77 pad 1: Row 5 -> Row 4
- D78 pad 1: Row 5 -> Row 4
- D79 pad 1: Row 5 -> Row 4
- D80 pad 1: Row 5 -> Row 4
- D85 pad 1: Row 6 -> Row 5
- D86 pad 1: Row 6 -> Row 5
- D87 pad 1: Row 6 -> Row 5
- D88 pad 1: Row 6 -> Row 5
- D89 pad 1: Row 6 -> Row 5
- D90 pad 1: Row 6 -> Row 5
- D91 pad 1: Row 6 -> Row 5
- D92 pad 1: Row 6 -> Row 5
- D93 pad 1: Row 6 -> Row 5
- D94 pad 1: Row 6 -> Row 5
- D95 pad 1: Row 6 -> Row 5
- D96 pad 1: Row 6 -> Row 5
- D99 pad 1: Row 7 -> Row 6
- S100 pad 1: Col 1 -> Col 3
- S101 pad 1: Col 2 -> Col 4
- S102 pad 1: Col 3 -> Col 5
- S103 pad 1: Col 4 -> Col 6
- S104 pad 1: Col 5 -> Col 7
- S105 pad 1: Col 6 -> Col 8
- S106 pad 1: Col 7 -> Col 9
- S107 pad 1: Col 8 -> Col 10
- S108 pad 1: Col 9 -> Col 11
- S109 pad 1: Col 10 -> Col 12
- S110 pad 1: Col 11 -> Col 13
- S111 pad 1: Col 12 -> Col 14
- S112 pad 1: Col 13 -> Col 15
- S15 pad 1: Col 0 -> Col 14
- S16 pad 1: Col 1 -> unconnected-(S16-Pad1)
- S17 pad 1: Col 2 -> Col 0
- S18 pad 1: Col 3 -> Col 1
- S19 pad 1: Col 4 -> Col 2
- S20 pad 1: Col 5 -> Col 3
- S21 pad 1: Col 6 -> Col 4
- S22 pad 1: Col 7 -> Col 5
- S23 pad 1: Col 8 -> Col 6
- S24 pad 1: Col 9 -> Col 7
- S25 pad 1: Col 10 -> Col 8
- S26 pad 1: Col 11 -> Col 9
- S27 pad 1: Col 12 -> unconnected-(S27-Pad1)
- S28 pad 1: Col 13 -> unconnected-(S28-Pad1)
- S29 pad 1: Col 0 -> Col 12
- S30 pad 1: Col 1 -> Col 13
- S31 pad 1: Col 2 -> Col 14
- S32 pad 1: Col 3 -> Col 15
- S33 pad 1: Col 4 -> Col 0
- S34 pad 1: Col 5 -> Col 1
- S35 pad 1: Col 6 -> Col 2
- S36 pad 1: Col 7 -> Col 3
- S37 pad 1: Col 8 -> Col 4
- S38 pad 1: Col 9 -> Col 5
- S39 pad 1: Col 10 -> Col 6
- S40 pad 1: Col 11 -> Col 7
- S41 pad 1: Col 12 -> Col 8
- S42 pad 1: Col 13 -> Col 9
- S43 pad 1: Col 0 -> Col 10
- S44 pad 1: Col 1 -> Col 11
- S45 pad 1: Col 2 -> Col 12
- S46 pad 1: Col 3 -> Col 13
- S47 pad 1: Col 4 -> Col 14
- S48 pad 1: Col 5 -> Col 15
- S49 pad 1: Col 6 -> Col 0
- S50 pad 1: Col 7 -> Col 1
- S51 pad 1: Col 8 -> Col 2
- S52 pad 1: Col 9 -> Col 3
- S53 pad 1: Col 10 -> Col 4
- S54 pad 1: Col 11 -> Col 5
- S55 pad 1: Col 12 -> Col 6
- S56 pad 1: Col 13 -> Col 7
- S57 pad 1: Col 0 -> Col 8
- S58 pad 1: Col 1 -> Col 9
- S59 pad 1: Col 2 -> Col 10
- S60 pad 1: Col 3 -> Col 11
- S61 pad 1: Col 4 -> Col 12
- S62 pad 1: Col 5 -> Col 13
- S63 pad 1: Col 6 -> Col 14
- S64 pad 1: Col 7 -> Col 15
- S65 pad 1: Col 8 -> Col 0
- S66 pad 1: Col 9 -> Col 1
- S67 pad 1: Col 10 -> Col 2
- S68 pad 1: Col 11 -> Col 3
- S69 pad 1: Col 12 -> Col 4
- S70 pad 1: Col 13 -> Col 5
- S71 pad 1: Col 0 -> Col 6
- S72 pad 1: Col 1 -> Col 7
- S73 pad 1: Col 2 -> Col 8
- S74 pad 1: Col 3 -> Col 9
- S75 pad 1: Col 4 -> Col 10
- S76 pad 1: Col 5 -> Col 11
- S77 pad 1: Col 6 -> Col 12
- S78 pad 1: Col 7 -> Col 13
- S79 pad 1: Col 8 -> Col 14
- S80 pad 1: Col 9 -> Col 15
- S81 pad 1: Col 10 -> Col 0
- S82 pad 1: Col 11 -> Col 1
- S83 pad 1: Col 12 -> Col 2
- S84 pad 1: Col 13 -> Col 3
- S85 pad 1: Col 0 -> Col 4
- S86 pad 1: Col 1 -> Col 5
- S87 pad 1: Col 2 -> Col 6
- S88 pad 1: Col 3 -> Col 7
- S89 pad 1: Col 4 -> Col 8
- S90 pad 1: Col 5 -> Col 9
- S91 pad 1: Col 6 -> Col 10
- S92 pad 1: Col 7 -> Col 11
- S93 pad 1: Col 8 -> Col 12
- S94 pad 1: Col 9 -> Col 13
- S95 pad 1: Col 10 -> Col 14
- S96 pad 1: Col 11 -> Col 15
- S97 pad 1: Col 12 -> Col 0
- S98 pad 1: Col 13 -> Col 1
- S99 pad 1: Col 0 -> Col 2
- U1 pad 12: Row 7 -> unconnected-(U1-D9-Pad12)
- U1 pad 15: NANO_MUX 6 -> unconnected-(U1-D14-Pad15)
- U1 pad 16: NANO_MUX 5 -> unconnected-(U1-D15-Pad16)
- U1 pad 21: +3.3V -> HIGH
Routing:
- net (no net): vias 0 -> 1

Commit message: minors
Parts:
- removed D111, D112, D31, D32, D79, D80, D95, D96: Diode, ScottoKeebs_Components:Diode_SOD-123
- removed S111: PAD7, ScottoKeebs_MX:MX_PCB_1.00u
- removed S112: PAD8, ScottoKeebs_MX:MX_PCB_1.00u
- removed S31: PAD1, ScottoKeebs_MX:MX_PCB_1.00u
- removed S32: PAD2, ScottoKeebs_MX:MX_PCB_1.00u
- removed S79: PAD3, ScottoKeebs_MX:MX_PCB_1.00u
- removed S80: PAD4, ScottoKeebs_MX:MX_PCB_1.00u
- removed S95: PAD5, ScottoKeebs_MX:MX_PCB_1.00u
- removed S96: PAD6, ScottoKeebs_MX:MX_PCB_1.00u
- U5: moved to B.Cu
- moved U5 179.9 mm to (390.8, 45.6)
- moved U1 161.4 mm to (407.5, 38.4)
- moved D81 12.6 mm to (55.1, 155.8)
- moved D82 12.6 mm to (78.9, 155.8)
- moved D83 12.6 mm to (102.7, 155.8)
- moved D84 12.6 mm to (174.1, 155.8)
- moved D85 12.6 mm to (245.6, 155.8)
- moved D86 12.6 mm to (269.4, 155.8)
- moved D87 12.6 mm to (293.2, 155.8)
- moved D88 12.6 mm to (317.0, 155.8)
- moved D89 12.6 mm to (343.2, 155.8)
- moved D90 12.6 mm to (362.3, 155.8)
- moved D91 12.6 mm to (381.3, 155.8)
- moved D92 12.6 mm to (421.8, 155.8)
- moved D93 12.6 mm to (443.2, 155.8)
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Connections:
- S110 pad 1: Col 13 -> unconnected-(S110-Pad1)
Routing:
- net Row 5: track 0.00 -> 411.1 mm
- net Row 3: track 0.00 -> 346.0 mm
- net Row 0: track 0.00 -> 328.6 mm
- net Row 6: track 0.00 -> 318.9 mm
- net Row 4: track 0.00 -> 304.8 mm
- net Col 3: track 0.00 -> 272.7 mm, vias 0 -> 1
- net Row 1: track 0.00 -> 264.3 mm
- net Col 13: track 0.00 -> 239.9 mm
- net Row 2: track 0.00 -> 233.4 mm
- net Col 2: track 0.00 -> 186.8 mm
- net Col 1: track 0.00 -> 167.0 mm, vias 0 -> 1
- net Col 4: track 0.00 -> 151.6 mm, vias 0 -> 1
- net Col 0: track 0.00 -> 141.7 mm, vias 0 -> 1
- net Col 12: track 0.00 -> 138.8 mm
- net Col 9: track 0.00 -> 116.9 mm
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
Commit message: update schema
Parts:
- added D12: Diode, ScottoKeebs_Components:Diode_SOD-123, F.Cu at (493.8, 60.6)
- added S12: F11, ScottoKeebs_MX:MX_PCB_1.00u, F.Cu at (501.0, 48.9)
Connections:
- S110 pad 1: unconnected-(S110-Pad1) -> Col 13
- S27 pad 1: unconnected-(S27-Pad1) -> Col 10
- S28 pad 1: unconnected-(S28-Pad1) -> Col 11

Commit message: pcb and schematic v1.0b
Parts:
- removed the D12 at (300.4, 51.1)
- removed the S12 at (290.8, 43.2)
- added D31: Diode, ScottoKeebs_Components:Diode_SOD-123, B.Cu at (295.8, 118.6)
- added D32: BLOC SCORR, LED_THT:LED_D3.0mm, F.Cu at (449.2, 31.4)
- added D79: CAPS LOCK, LED_THT:LED_D3.0mm, F.Cu at (437.0, 31.4)
- added D80: BLOC NUM, LED_THT:LED_D3.0mm, F.Cu at (443.1, 31.4)
- added D95: MIC ON, LED_THT:LED_D3.0mm, F.Cu at (455.3, 31.4)
- added D96: AUDIO ON, LED_THT:LED_D3.0mm, F.Cu at (461.4, 31.4)
- added R1: 180, Resistor_THT:R_Axial_DIN0204_L3.6mm_D1.6mm_P7.62mm_Horizontal, F.Cu at (442.8, 40.3)
- added R2: 180, Resistor_THT:R_Axial_DIN0204_L3.6mm_D1.6mm_P7.62mm_Horizontal, F.Cu at (442.8, 54.5)
- added R3: 180, Resistor_THT:R_Axial_DIN0204_L3.6mm_D1.6mm_P7.62mm_Horizontal, F.Cu at (442.8, 43.8)
- added R4: 180, Resistor_THT:R_Axial_DIN0204_L3.6mm_D1.6mm_P7.62mm_Horizontal, F.Cu at (442.8, 47.4)
- added R5: 180, Resistor_THT:R_Axial_DIN0204_L3.6mm_D1.6mm_P7.62mm_Horizontal, F.Cu at (442.8, 50.9)
- added REF**: MountingHole_3.2mm_M3, MountingHole:MountingHole_3.2mm_M3, F.Cu at (173.5, 166.5)
- added REF**: MountingHole_3.2mm_M3, MountingHole:MountingHole_3.2mm_M3, F.Cu at (471.3, 166.5)
- added REF**: MountingHole_3.2mm_M3, MountingHole:MountingHole_3.2mm_M3, F.Cu at (322.4, 166.5)
- added REF**: MountingHole_3.2mm_M3, MountingHole:MountingHole_3.2mm_M3, F.Cu at (173.5, 24.6)
- added REF**: MountingHole_3.2mm_M3, MountingHole:MountingHole_3.2mm_M3, F.Cu at (322.4, 24.7)
- added REF**: MountingHole_3.2mm_M3, MountingHole:MountingHole_3.2mm_M3, F.Cu at (24.6, 24.6)
- added REF**: MountingHole_3.2mm_M3, MountingHole:MountingHole_3.2mm_M3, F.Cu at (471.3, 24.6)
- added REF**: MountingHole_3.2mm_M3, MountingHole:MountingHole_3.2mm_M3, F.Cu at (24.6, 166.5)
- added S31: ù, ScottoKeebs_Hotswap:Hotswap_MX_Plated, F.Cu at (286.1, 110.0)
- added U2: 4052, Package_SO:TSSOP-16-1EP_4.4x5mm_P0.65mm_EP3x3mm, B.Cu at (428.9, 36.0)
- D12: moved to B.Cu
- S1, S10, S100, S101, S102, S103, S104, S105, S106, S107, S108, S109, S11, S110, S12, S13, S14, S15, S16, S17, S18, S19, S2, S20, S21, S22, S23, S24, S25, S26, S27, S28, S29, S3, S30, S33, S34, S35, S36, S37, S38, S39, S4, S40, S41, S42, S43, S44, S45, S46, S47, S48, S49, S5, S50, S51, S52, S53, S54, S55, S56, S57, S58, S59, S6, S60, S61, S62, S63, S64, S65, S66, S67, S68, S69, S7, S70, S71, S72, S73, S74, S75, S76, S77, S78, S8, S81, S82, S83, S84, S85, S86, S87, S88, S89, S9, S90, S91, S92, S93, S94, S97, S98, S99: footprint ScottoKeebs_MX:MX_PCB_1.00u -> ScottoKeebs_Hotswap:Hotswap_MX_Plated
- moved S12 210.3 mm to (290.8, 43.2)
- moved D12 193.7 mm to (300.4, 51.1), turned to 90 degrees
- moved U5 7.53 mm to (398.0, 47.9), turned to 180 degrees
- moved U1 7.03 mm to (414.5, 38.6)
- moved D110 1.65 mm to (441.6, 136.8)
- moved D103 1.14 mm to (442.1, 98.7)
- moved D78 0.98 mm to (362.2, 135.8)
Connections:
- D100 pad 1: Row 6 -> Row 0
- D101 pad 1: Row 6 -> Row 1
- D102 pad 1: Row 6 -> Row 1
- D103 pad 1: Row 6 -> Row 1
- D104 pad 1: Row 6 -> Row 1
- D105 pad 1: Row 6 -> Row 2
- D106 pad 1: Row 6 -> Row 2
- D107 pad 1: Row 6 -> Row 2
- D108 pad 1: Row 6 -> Row 3
- D109 pad 1: Row 6 -> Row 3
- D110 pad 1: Row 6 -> Row 3
- D12 pad 1: Row 1 -> Row 0
- D85 pad 1: Row 5 -> Row 6
- D86 pad 1: Row 5 -> Row 6
- D87 pad 1: Row 5 -> Row 6
- D88 pad 1: Row 5 -> Row 6
- D89 pad 1: Row 5 -> Row 6
- D90 pad 1: Row 5 -> Row 6
- D92 pad 1: Row 5 -> Row 4
- D93 pad 1: Row 5 -> Row 4
- D94 pad 1: Row 5 -> Row 4
- D97 pad 1: Row 6 -> Row 0
- D98 pad 1: Row 6 -> Row 0
- D99 pad 1: Row 6 -> Row 0
- S100 pad 1: Col 3 -> Pad Col 3
- S101 pad 1: Col 4 -> Pad Col 0
- S102 pad 1: Col 5 -> Pad Col 1
- S103 pad 1: Col 6 -> Pad Col 2
- S104 pad 1: Col 7 -> Pad Col 3
- S105 pad 1: Col 8 -> Pad Col 0
- S106 pad 1: Col 9 -> Pad Col 1
- S107 pad 1: Col 10 -> Pad Col 2
- S108 pad 1: Col 11 -> Pad Col 0
- S109 pad 1: Col 12 -> Pad Col 1
- S110 pad 1: Col 13 -> Pad Col 2
- S12 pad 1: Col 14 -> Col 11
- S16 pad 1: unconnected-(S16-Pad1) -> Col 15
- S78 pad 1: Col 13 -> Col 15
- S85 pad 1: Col 4 -> Col 8
- S86 pad 1: Col 5 -> Col 9
- S87 pad 1: Col 6 -> Col 10
- S88 pad 1: Col 7 -> Col 11
- S89 pad 1: Col 8 -> Col 13
- S90 pad 1: Col 9 -> Col 14
- S92 pad 1: Col 11 -> Pad Col 0
- S93 pad 1: Col 12 -> Pad Col 2
- S94 pad 1: Col 13 -> Pad Col 3
- S97 pad 1: Col 0 -> Pad Col 0
- S98 pad 1: Col 1 -> Pad Col 1
- S99 pad 1: Col 2 -> Pad Col 2
- U1 pad 1: unconnected-(U1-D1-Pad1) -> LED_MUX 1
- U1 pad 10: Row 5 -> Row 1
- U1 pad 11: Row 6 -> Row 0
- U1 pad 13: unconnected-(U1-D10-Pad13) -> Pad Col 0
- U1 pad 14: unconnected-(U1-D16-Pad14) -> Pad Col 1
- U1 pad 15: unconnected-(U1-D14-Pad15) -> Pad Col 2
- U1 pad 16: unconnected-(U1-D15-Pad16) -> Pad Col 3
- U1 pad 2: unconnected-(U1-D0-Pad2) -> LED_MUX 2
- U1 pad 5: Row 0 -> Row 6
- U1 pad 6: Row 1 -> Row 5
- U1 pad 7: Row 2 -> Row 4
- U1 pad 9: Row 4 -> Row 2
- U5 pad 10: NANO_MUX 2 -> NANO_MUX 1
- U5 pad 11: NANO_MUX 1 -> NANO_MUX 2
- U5 pad 16: Col 15 -> Col 7
- U5 pad 17: Col 14 -> Col 6
- U5 pad 18: Col 13 -> Col 5
- U5 pad 19: Col 12 -> Col 4
- U5 pad 2: Col 7 -> Col 8
- U5 pad 20: Col 11 -> Col 3
- U5 pad 21: Col 10 -> Col 2
- U5 pad 22: Col 9 -> Col 1
- U5 pad 23: Col 8 -> Col 0
- U5 pad 3: Col 6 -> Col 9
- U5 pad 4: Col 5 -> Col 10
- U5 pad 5: Col 4 -> Col 11
- U5 pad 6: Col 3 -> Col 12
- U5 pad 7: Col 2 -> Col 13
- U5 pad 8: Col 1 -> Col 14
- U5 pad 9: Col 0 -> Col 15
Routing:
- net Row 2: track 233.4 -> 574.4 mm
- net Col 0: track 141.7 -> 475.3 mm
- net Col 10: track 107.4 -> 437.2 mm, vias 0 -> 1
- net Col 1: track 167.0 -> 465.7 mm
- net Row 4: track 304.8 -> 587.9 mm
- net Row 1: track 264.3 -> 546.1 mm
- net Row 3: track 346.0 -> 608.4 mm
- net Col 8: track 108.5 -> 368.7 mm, vias 0 -> 1
- net Col 5: track 108.5 -> 363.3 mm, vias 0 -> 1
- net Col 2: track 186.8 -> 436.2 mm, vias 0 -> 1
- net Col 6: track 108.5 -> 344.6 mm, vias 0 -> 1
- net Col 9: track 116.9 -> 347.9 mm, vias 0 -> 1
- net Row 5: track 411.1 -> 639.4 mm, vias 0 -> 2
- net Col 4: track 151.6 -> 375.5 mm
- net Col 7: track 108.5 -> 328.6 mm, vias 0 -> 1
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Other:
- board outline added: 454.6 x 149.8 mm
- board text added: "K3yb it! designed by Andrea Novati la tastiera perfetta non esist... v1.0b"
