File: k3yb.it/k3yb.it.kicad_pcb (KiCad board)
At the start: 2 copper layers, 454.6 x 149.8 mm, 229 parts, among them U1 Nice_Nano_V2, U2 4052, U5 CD74HC4067M

Commit message: added Gerber fixed led output multiplexing
Connections:
- U2 pad 11: LED_OUTPUT -> HIGH
- U2 pad 12: LED_OUTPUT -> HIGH
- U2 pad 13: HIGH -> Net-(U2-X)
- U2 pad 14: LED_OUTPUT -> HIGH
- U2 pad 15: LED_OUTPUT -> HIGH
- U2 pad 3: HIGH -> Net-(U2-X)
- U2 pad 6: LOW -> LED_OUTPUT
Routing:
- net LOW: track 122.8 -> 130.7 mm
- net LED_OUTPUT: track 34.8 -> 42.4 mm
- net Net-(U2-X): track 0.00 -> 7.03 mm
- net Net-(D76-A): track 16.7 -> 22.9 mm
- net Net-(D30-A): track 23.9 -> 27.3 mm
- net Row 3: track 608.4 -> 606.0 mm
- net HIGH: track 49.5 -> 47.5 mm
- net Net-(D84-A): track 16.7 -> 18.1 mm
- net Net-(D27-A): track 16.7 -> 18.1 mm
- net Net-(D21-A): track 16.7 -> 18.1 mm
- net Net-(D19-A): track 16.7 -> 18.1 mm
- net Net-(D25-A): track 16.7 -> 18.1 mm
- net Net-(D104-A): track 16.7 -> 18.1 mm
- net Net-(D33-A): track 16.7 -> 18.1 mm
- net Net-(D78-A): track 15.8 -> 17.2 mm
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
Commit message: added user drawings
Parts:
- renumbered REF** to M3
Changed lines of the file:
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@@
     (tags "mounting hole 3.2mm no annular m3")
     (attr exclude_from_pos_files exclude_from_bom)
-    (fp_text reference "REF**" (at 6.1391 -0.310966) (layer "F.SilkS")
+    (fp_text reference "M3" (at 6.1391 -0.310966) (layer "F.SilkS")
         (effects (font (size 1 1) (thickness 0.15)))
     )
@@
     (tags "mounting hole 3.2mm no annular m3")
     (attr exclude_from_pos_files exclude_from_bom)
-    (fp_text reference "REF**" (at -6.115611 0.177632) (layer "F.SilkS")
+    (fp_text reference "M3" (at -6.115611 0.177632) (layer "F.SilkS")
         (effects (font (size 1 1) (thickness 0.15)))
     )
@@
     (tags "mounting hole 3.2mm no annular m3")
     (attr exclude_from_pos_files exclude_from_bom)
-    (fp_text reference "REF**" (at 5.774408 -0.322368) (layer "F.SilkS")
+    (fp_text reference "M3" (at 5.774408 -0.322368) (layer "F.SilkS")
         (effects (font (size 1 1) (thickness 0.15)))
     )
@@
     (tags "mounting hole 3.2mm no annular m3")
     (attr exclude_from_pos_files exclude_from_bom)
-    (fp_text reference "REF**" (at 5.654325 0.008428) (layer "F.SilkS")
+    (fp_text reference "M3" (at 5.654325 0.008428) (layer "F.SilkS")
         (effects (font (size 1 1) (thickness 0.15)))
     )
@@
     (tags "mounting hole 3.2mm no annular m3")
     (attr exclude_from_pos_files exclude_from_bom)
-    (fp_text reference "REF**" (at 5.766823 0.000843) (layer "F.SilkS")
+    (fp_text reference "M3" (at 5.766823 0.000843) (layer "F.SilkS")
         (effects (font (size 1 1) (thickness 0.15)))
     )
@@
     (tags "mounting hole 3.2mm no annular m3")
     (attr exclude_from_pos_files exclude_from_bom)
-    (fp_text reference "REF**" (at 6.029987 0.029987) (layer "F.SilkS")
+    (fp_text reference "M3" (at 6.029987 0.029987) (layer "F.SilkS")
         (effects (font (size 1 1) (thickness 0.15)))
     )
@@
     (tags "mounting hole 3.2mm no annular m3")
     (attr exclude_from_pos_files exclude_from_bom)
-    (fp_text reference "REF**" (at -6.114767 0.007185) (layer "F.SilkS")
+    (fp_text reference "M3" (at -6.114767 0.007185) (layer "F.SilkS")
         (effects (font (size 1 1) (thickness 0.15)))
     )
@@
     (tags "mounting hole 3.2mm no annular m3")
     (attr exclude_from_pos_files exclude_from_bom)
-    (fp_text reference "REF**" (at 6.012387 -0.318323) (layer "F.SilkS")
+    (fp_text reference "M3" (at 6.012387 -0.318323) (layer "F.SilkS")
         (effects (font (size 1 1) (thickness 0.15)))
     )
