File: k3yb.it/k3yb.it.kicad_pcb (KiCad board)
At the start: 2 copper layers, 454.6 x 149.8 mm, 229 parts, among them M3 MountingHole_3.2mm_M3, U1 Nice_Nano_V2, U2 4052, U5 CD74HC4067M

Commit message: added stabilizer mounting holes
Parts:
- added REF**: Stabilizer_MX_2.00u, ScottoKeebs_Stabilizer:Stabilizer_MX_2.00u, F.Cu at (451.7, 138.4)
- added REF**: Stabilizer_MX_2.00u, ScottoKeebs_Stabilizer:Stabilizer_MX_2.00u, F.Cu at (306.4, 100.4)
- added REF**: Stabilizer_MX_2.00u, ScottoKeebs_Stabilizer:Stabilizer_MX_2.00u, F.Cu at (405.2, 149.0)
- added REF**: Stabilizer_MX_2.00u, ScottoKeebs_Stabilizer:Stabilizer_MX_2.00u, F.Cu at (293.2, 130.0)
- added REF**: Stabilizer_MX_2.00u, ScottoKeebs_Stabilizer:Stabilizer_MX_2.00u, F.Cu at (300.4, 72.8)
- added REF**: Stabilizer_MX_6.25u, ScottoKeebs_Stabilizer:Stabilizer_MX_6.25u, F.Cu at (164.6, 149.0)
- added REF**: Stabilizer_MX_2.00u, ScottoKeebs_Stabilizer:Stabilizer_MX_2.00u, F.Cu at (451.5, 100.3)
- moved D68 0.89 mm to (114.6, 135.9)
Routing:
- net Row 5: track 639.4 -> 648.0 mm
- net Net-(D30-A): track 27.3 -> 31.2 mm
- net Row 3: track 606.0 -> 603.0 mm
- net Net-(D110-A): track 18.6 -> 16.4 mm
- net Col 3: track 462.9 -> 464.9 mm
- net Net-(D103-A): track 18.4 -> 16.5 mm
- net Row 2: track 574.4 -> 576.0 mm
- net Row 1: track 546.1 -> 547.6 mm
- net Net-(D93-A): track 17.8 -> 16.8 mm
- net Net-(D68-A): track 17.6 -> 16.7 mm
- net Row 4: track 587.9 -> 587.1 mm
- net Net-(D107-A): track 18.0 -> 17.4 mm
- net Col 14: track 173.5 -> 172.9 mm

Commit message: added dxf, added reset switch
Parts:
- added SW1: Nice!Nano Reset, Button_Switch_THT:SW_PUSH_1P1T_6x3.5mm_H4.3_APEM_MJTP1243, F.Cu at (427.7, 46.2)
Routing:
- net NANO_RST: track 0.00 -> 26.1 mm, vias 0 -> 2
- net LOW: track 130.7 -> 134.0 mm
Changed lines of the file:
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@@
     )
   )
+  (footprint "Button_Switch_THT:SW_PUSH_1P1T_6x3.5mm_H4.3_APEM_MJTP1243" (layer "F.Cu")
+    (at 427.655 46.155 -90)
+    (descr "tactile push button, 6x3.5mm, https://www.apem.com/idec-apem/en_US/PCB-switches/Tactile-Switches/MJTP-6mm-through-hole/c/MJTP_6mm_through%20hole?page=1")
+    (tags "PHAP3362 6mm tact sw THT")
+    (property "Sheetfile" "k3yb.it.kicad_sch")
+    (property "Sheetname" "")
+    (property "ki_description" "Push button switch, generic, separate symbols, four pins")
+    (property "ki_keywords" "switch normally-open pushbutton push-button")
+    (attr through_hole)
+    (fp_text reference "SW1" (at 3.42 -2.7 90) (layer "F.SilkS")
+        (effects (font (size 1 1) (thickness 0.15)))
+    )
+    (fp_text value "Nice!Nano Reset" (at 4.4 3.7 90) (layer "F.Fab")
+        (effects (font (size 1 1) (thickness 0.15)))
+    )
+    (fp_text user "${REFERENCE}" (at 3 0 90) (layer "F.Fab")
+        (effects (font (size 1 1) (thickness 0.15)))
+    )
+    (fp_line (start 0.15 -1.85) (end 0.15 -1.39)
+      (stroke (width 0.12) (type default)) (layer "F.SilkS"))
+    (fp_line (start 0.15 -1.39) (end -0.85 -1.39)
+      (stroke (width 0.12) (type default)) (layer "F.SilkS"))
+    (fp_line (start 0.15 1.39) (end 0.15 1.85)
+      (stroke (width 0.12) (type solid)) (layer "F.SilkS"))
+    (fp_line (start 0.15 1.85) (end 6.35 1.85)
+      (stroke (width 0.12) (type solid)) (layer "F.SilkS"))
+    (fp_line (start 6.35 -1.85) (end 0.15 -1.85)
+      (stroke (width 0.12) (type solid)) (layer "F.SilkS"))
+    (fp_line (start 6.35 -1.85) (end 6.35 -1.39)
+      (stroke (width 0.12) (type solid)) (layer "F.SilkS"))
+    (fp_line (start 6.35 1.39) (end 6.35 1.85)
+      (stroke (width 0.12) (type solid)) (layer "F.SilkS"))
+    (fp_rect (start 1.75 -0.55) (end 4.6 0.5)
+      (stroke (width 0.12) (type default)) (fill none) (layer "F.SilkS"))
+    (fp_line (start -1.38 -1.38) (end 0 -1.38)
+      (stroke (width 0.05) (type default)) (layer "F.CrtYd"))
+    (fp_line (start -1.38 1.38) (end -1.38 -1.38)
+      (stroke (width 0.05) (type solid)) (layer "F.CrtYd"))
+    (fp_line (start -1.38 1.38) (end 0 1.38)
+      (stroke (width 0.05) (type default)) (layer "F.CrtYd"))
+    (fp_line (start 0 -2) (end 0 -1.38)
+      (stroke (width 0.05) (type default)) (layer "F.CrtYd"))
+    (fp_line (start 0 -2) (end 6.5 -2)
+      (stroke (width 0.05) (type solid)) (layer "F.CrtYd"))
+    (fp_line (start 0 1.38) (end 0 2)
+      (stroke (width 0.05) (type default)) (layer "F.CrtYd"))
+    (fp_line (start 6.5 -2) (end 6.5 -1.38)
+      (stroke (width 0.05) (type default)) (layer "F.CrtYd"))
+    (fp_line (start 6.5 1.38) (end 6.5 2)
+      (stroke (width 0.05) (type default)) (layer "F.CrtYd"))
+    (fp_line (start 6.5 2) (end 0 2)
+      (stroke (width 0.05) (type solid)) (layer "F.CrtYd"))
+    (fp_arc (start 6.5 -1.38) (mid 7.88 0) (end 6.5 1.38)
+      (stroke (width 0.05) (type default)) (layer "F.CrtYd"))
+    (fp_line (start 0.25 1.75) (end 0.25 -1.35)
+      (stroke (width 0.1) (type solid)) (layer "F.Fab"))
+    (fp_line (start 0.65 -1.75) (end 0.25 -1.35)
+      (stroke (width 0.1) (type default)) (layer "F.Fab"))
+    (fp_line (start 0.65 -1.75) (end 6.25 -1.75)
+      (stroke (width 0.1) (type solid)) (layer "F.Fab"))
+    (fp_line (start 6.25 -1.75) (end 6.25 1.75)
+      (stroke (width 0.1) (type solid)) (layer "F.Fab"))
+    (fp_line (start 6.25 1.75) (end 0.25 1.75)
+      (stroke (width 0.1) (type solid)) (layer "F.Fab"))
+    (pad "1" thru_hole rect (at 0 0) (size 2.25 2.25) (drill 1.3) (layers "*.Cu" "*.Mask")
+      (net 1 "LOW") (pinfunction "C") (pintype "passive"))
+    (pad "2" thru_hole circle (at 6.5 0) (size 2.25 2.25) (drill 1.3) (layers "*.Cu" "*.Mask")
+      (net 125 "NANO_RST") (pinfunction "D") (pintype "passive"))
+    (model "${KICAD7_3DMODEL_DIR}/Button_Switch_THT.3dshapes/SW_PUSH_1P1T_6x3.5mm_H4.3_APEM_MJTP1243.wrl"
+      (offset (xyz 0 0 0))
+      (scale (xyz 1 1 1))
+      (rotate (xyz 0 0 0))
+    )
+  )
   (footprint "ScottoKeebs_Hotswap:Hotswap_MX_Plated" (layer "F.Cu")
     (at 138.43 71.755)
@@
   )
   (segment (start 431.927 43.815) (end 429.895 43.815) (width 0.25) (layer "F.Cu") (net 1))
+  (segment (start 429.895 43.915) (end 427.655 46.155) (width 0.25) (layer "F.Cu") (net 1))
+  (segment (start 429.895 43.815) (end 429.895 43.915) (width 0.25) (layer "F.Cu") (net 1))
   (segment (start 429.895 43.815) (end 429.155 43.075) (width 0.25) (layer "F.Cu") (net 1))
   (segment (start 429.155 43.075) (end 429.155 29.155) (width 0.25) (layer "F.Cu") (net 1))
@@
   (segment (start 428.879 43.815) (end 429.895 42.799) (width 0.25) (layer "B.Cu") (net 124))
   (segment (start 429.895 42.799) (end 429.895 38.227) (width 0.25) (layer "B.Cu") (net 124))
+  (segment (start 427.655 52.655) (end 427.655 49.155) (width 0.25) (layer "F.Cu") (net 125))
+  (segment (start 424.155 45.655) (end 424.155 43.655) (width 0.25) (layer "F.Cu") (net 125))
+  (segment (start 424.155 30.655) (end 423.235 29.735) (width 0.25) (layer "F.Cu") (net 125))
+  (segment (start 424.155 32.155) (end 424.155 30.655) (width 0.25) (layer "F.Cu") (net 125))
+  (segment (start 427.655 49.155) (end 424.155 45.655) (width 0.25) (layer "F.Cu") (net 125))
+  (segment (start 423.235 29.735) (end 422.155 29.735) (width 0.25) (layer "F.Cu") (net 125))
+  (via (at 424.155 43.655) (size 0.8) (drill 0.4) (layers "F.Cu" "B.Cu") (net 125))
+  (via (at 424.155 32.155) (size 0.8) (drill 0.4) (layers "F.Cu" "B.Cu") (net 125))
+  (segment (start 423.857 43.357) (end 423.857 32.453) (width 0.25) (layer "B.Cu") (net 125))
+  (segment (start 424.155 43.655) (end 423.857 43.357) (width 0.25) (layer "B.Cu") (net 125))
+  (segment (start 423.857 32.453) (end 424.155 32.155) (width 0.25) (layer "B.Cu") (net 125))
   (segment (start 436.91175 126.52375) (end 436.245 125.857) (width 0.25) (layer "F.Cu") (net 127))
   (segment (start 436.245 125.857) (end 436.245 123.825) (width 0.25) (layer "F.Cu") (net 127))
