File: k3yb.it/k3yb.it.kicad_sch (KiCad schematic)
At the start: 228 parts, among them U1 Nice_Nano_V2, U2 4052, U3 4052, U4 4052

Commit message: alligned component Soldering MX version
Parts:
- removed U2, U3, U4: 4052, Package_SO:SO-16_3.9x9.9mm_P1.27mm, symbol 4xxx:4052
- added U5: CD74HC4067M, Package_SO:SOIC-24W_7.5x15.4mm_P1.27mm, symbol 74xx:CD74HC4067M
- D1: footprint ScottoKeebs_Hotswap:Hotswap_Choc_V1V2_1.00u -> ScottoKeebs_Components:Diode_SOD-123
- S1: value Keyswitch -> Esc
- S10: value Keyswitch -> F9
- S100, S28: value Keyswitch -> -
- S101, S24: value Keyswitch -> 7
- S102, S25: value Keyswitch -> 8
- S103, S26: value Keyswitch -> 9
- S104: value Keyswitch -> +
- S105, S21: value Keyswitch -> 4
- S106, S22: value Keyswitch -> 5
- S107, S23: value Keyswitch -> 6
- S108, S18: value Keyswitch -> 1
- S109, S19: value Keyswitch -> 2
- S11: value Keyswitch -> F10
- S110, S20: value Keyswitch -> 3
- S111: value Keyswitch -> PAD7
- S112: value Keyswitch -> PAD8
- S12: value Keyswitch -> F11
- S13: value Keyswitch -> F12
- S14: value Keyswitch -> Stamp
- S15: value Keyswitch -> Bloc scorr
- S16: value Keyswitch -> Pause
- S17: value Keyswitch -> tilde
- S2: value Keyswitch -> F1
- S27, S92: value Keyswitch -> 0
- S29: value Keyswitch -> =
- S3: value Keyswitch -> F2
- S30: value Keyswitch -> Backspace
- S31: value Keyswitch -> PAD1
- S32: value Keyswitch -> PAD2
- S33: value Keyswitch -> Tab
- S34: value Keyswitch -> q
- S35: value Keyswitch -> w
- S36: value Keyswitch -> e
- S37: value Keyswitch -> r
- S38: value Keyswitch -> t
- S39: value Keyswitch -> y
- S4: value Keyswitch -> F3
- S40: value Keyswitch -> u
- S41: value Keyswitch -> i
- S42: value Keyswitch -> o
- S43: value Keyswitch -> p
- S44: value Keyswitch -> {
- S45: value Keyswitch -> }
- S46: value Keyswitch -> ins
- S47, S78: value Keyswitch -> up
- S48: value Keyswitch -> pg up
- S49: value Keyswitch -> Caps lock
- S5: value Keyswitch -> F4
- S50: value Keyswitch -> a
- S51: value Keyswitch -> s
- S52: value Keyswitch -> d
- S53: value Keyswitch -> f
- S54: value Keyswitch -> g
- S55: value Keyswitch -> h
- S56: value Keyswitch -> j
- S57: value Keyswitch -> k
- S58: value Keyswitch -> l
- S59: value Keyswitch -> ;
- S6: value Keyswitch -> F5
- S60: value Keyswitch -> '
- S61, S94: value Keyswitch -> enter
- S62: value Keyswitch -> del
- S63: value Keyswitch -> end
- S64: value Keyswitch -> pg dowm
- S65: value Keyswitch -> Left Shift
- S66: value Keyswitch -> \
- S67: value Keyswitch -> z
- S68: value Keyswitch -> x
- S69: value Keyswitch -> c
- S7: value Keyswitch -> F6
- S70: value Keyswitch -> v
- S71: value Keyswitch -> b
- S72: value Keyswitch -> n
- S73: value Keyswitch -> m
- S74: value Keyswitch -> ,
- S75, S93: value Keyswitch -> .
- S76, S98: value Keyswitch -> /
- S77: value Keyswitch -> right shift
- S79: value Keyswitch -> PAD3
- S8: value Keyswitch -> F7
- S80: value Keyswitch -> PAD4
- S81: value Keyswitch -> left ctrl
- S82: value Keyswitch -> win
- S83: value Keyswitch -> left alt
- S84: value Keyswitch -> space
- S85: value Keyswitch -> right alt
- S86: value Keyswitch -> fn
- S87: value Keyswitch -> menu
- S88: value Keyswitch -> right ctrl
- S89: value Keyswitch -> left
- S9: value Keyswitch -> F8
- S90: value Keyswitch -> down
- S91: value Keyswitch -> right
- S95: value Keyswitch -> PAD5
- S96: value Keyswitch -> PAD6
- S97: value Keyswitch -> num
- S99: value Keyswitch -> *
Connections:
- net +3.3V: now also U5.24 (VCC)
- net Col 0: now also S17.1, S33.1, S49.1, S65.1, S81.1, S97.1, U5.9 (I0); no longer S15.1, S29.1, S43.1, S57.1, S71.1, S85.1, S99.1
- net Col 1: now also S18.1, S34.1, S50.1, S66.1, S82.1, S98.1, U5.8 (I1); no longer S100.1, S16.1, S30.1, S44.1, S58.1, S72.1, S86.1
- net Col 10: now also S107.1, S43.1, S59.1, S75.1, S91.1, U5.21 (I10); no longer S109.1, S25.1, S39.1, S53.1, S67.1, S81.1, S95.1
- net Col 11: now also S108.1, S44.1, S60.1, S76.1, S92.1, U5.20 (I11); no longer S110.1, S26.1, S40.1, S54.1, S68.1, S82.1, S96.1
- net Col 12: now also S109.1, S29.1, S45.1, S61.1, S77.1, S93.1, U5.19 (I12); no longer S111.1, S27.1, S41.1, S55.1, S69.1, S83.1, S97.1
- net Col 13: now also S110.1, S30.1, S46.1, S62.1, S78.1, S94.1, U5.18 (I13); no longer S112.1, S28.1, S42.1, S56.1, S70.1, S84.1, S98.1
- net Col 2: now also S19.1, S35.1, S51.1, S67.1, S83.1, S99.1, U5.7 (I2); no longer S101.1, S17.1, S31.1, S45.1, S59.1, S73.1, S87.1
- net Col 3: now also S100.1, S20.1, S36.1, S52.1, S68.1, S84.1, U5.6 (I3); no longer S102.1, S18.1, S32.1, S46.1, S60.1, S74.1, S88.1
- net Col 4: now also S101.1, S21.1, S37.1, S53.1, S69.1, S85.1, U5.5 (I4); no longer S103.1, S19.1, S33.1, S47.1, S61.1, S75.1, S89.1
- net Col 5: now also S102.1, S22.1, S38.1, S54.1, S70.1, S86.1, U5.4 (I5); no longer S104.1, S20.1, S34.1, S48.1, S62.1, S76.1, S90.1
- net Col 6: now also S103.1, S23.1, S39.1, S55.1, S71.1, S87.1, U5.3 (I6); no longer S105.1, S21.1, S35.1, S49.1, S63.1, S77.1, S91.1
- net Col 7: now also S104.1, S24.1, S40.1, S56.1, S72.1, S88.1, U5.2 (I7); no longer S106.1, S22.1, S36.1, S50.1, S64.1, S78.1, S92.1
- net Col 8: now also S105.1, S25.1, S41.1, S57.1, S73.1, S89.1, U5.23 (I8); no longer S107.1, S23.1, S37.1, S51.1, S65.1, S79.1, S93.1
- net Col 9: now also S106.1, S26.1, S42.1, S58.1, S74.1, S90.1, U5.22 (I9); no longer S108.1, S24.1, S38.1, S52.1, S66.1, S80.1, S94.1
- net GND: now also U5.1 (COM), U5.12 (GND), U5.15 (~{E})
- net NANO_MUX 1: now also U5.11 (S1)
- net NANO_MUX 2: now also U5.10 (S0)
- net NANO_MUX 3: now also U5.14 (S2)
- net NANO_MUX 4: now also U5.13 (S3)
- net Row 0: now also D15.1 (K), D16.1 (K)
- net Row 1: now also D29.1 (K), D30.1 (K), D31.1 (K), D32.1 (K); no longer D15.1 (K), D16.1 (K)
- net Row 2: now also D43.1 (K), D44.1 (K), D45.1 (K), D46.1 (K), D47.1 (K), D48.1 (K); no longer D29.1 (K), D30.1 (K), D31.1 (K), D32.1 (K)
- net Row 3: now also D57.1 (K), D58.1 (K), D59.1 (K), D60.1 (K), D61.1 (K), D62.1 (K), D63.1 (K), D64.1 (K); no longer D43.1 (K), D44.1 (K), D45.1 (K), D46.1 (K), D47.1 (K), D48.1 (K)
- net Row 4: now also D71.1 (K), D72.1 (K), D73.1 (K), D74.1 (K), D75.1 (K), D76.1 (K), D77.1 (K), D78.1 (K), D79.1 (K), D80.1 (K); no longer D57.1 (K), D58.1 (K), D59.1 (K), D60.1 (K), D61.1 (K), D62.1 (K), D63.1 (K), D64.1 (K)
- net Row 5: now also D85.1 (K), D86.1 (K), D87.1 (K), D88.1 (K), D89.1 (K), D90.1 (K), D91.1 (K), D92.1 (K), D93.1 (K), D94.1 (K), D95.1 (K), D96.1 (K); no longer D71.1 (K), D72.1 (K), D73.1 (K), D74.1 (K), D75.1 (K), D76.1 (K), D77.1 (K), D78.1 (K), D79.1 (K), D80.1 (K)
- net Row 6: now also D100.1 (K), D101.1 (K), D102.1 (K), D103.1 (K), D104.1 (K), D105.1 (K), D106.1 (K), D107.1 (K), D108.1 (K), D109.1 (K), D110.1 (K), D111.1 (K), D112.1 (K), D99.1 (K); no longer D85.1 (K), D86.1 (K), D87.1 (K), D88.1 (K), D89.1 (K), D90.1 (K), D91.1 (K), D92.1 (K), D93.1 (K), D94.1 (K), D95.1 (K), D96.1 (K)
- net NANO_MUX 5: no longer names the net of U1.16 (D15)
- net NANO_MUX 6: no longer names the net of U1.15 (D14)
- removed net Row 7: D100.1 (K), D101.1 (K), D102.1 (K), D103.1 (K), D104.1 (K), D105.1 (K), D106.1 (K), D107.1 (K), D108.1 (K), D109.1 (K), D110.1 (K), D111.1 (K), D112.1 (K), D99.1 (K), U1.12 (D9)
- new net Col 14: S111.1, S15.1, S31.1, S47.1, S63.1, S79.1, S95.1, U5.17 (I14)
- new net Col 15: S112.1, S32.1, S48.1, S64.1, S80.1, S96.1, U5.16 (I15)
- no-connect marks 11 -> 7
Other:
- note added: "MATRIX 112"
- note removed: "MAXTRIX 104"

Commit message: minors
Connections:
- net Col 13: no longer S110.1
- net Col 14: no longer S111.1, S31.1, S79.1, S95.1
- net Col 15: no longer S112.1, S32.1, S80.1, S96.1
- no-connect marks 7 -> 16
Other:
- moved on the sheet: D31, D32, S31, S32
Changed lines of the file:
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@@
   (junction (at 80.01 55.88) (diameter 0) (color 0 0 0 0)
   )
-  (junction (at 250.19 90.17) (diameter 0) (color 0 0 0 0)
-  )
   (junction (at 234.95 133.35) (diameter 0) (color 0 0 0 0)
   )
-  (junction (at 245.11 142.24) (diameter 0) (color 0 0 0 0)
-  )
   (junction (at 250.19 133.35) (diameter 0) (color 0 0 0 0)
   )
@@
   (junction (at 250.19 111.76) (diameter 0) (color 0 0 0 0)
   )
-  (junction (at 245.11 77.47) (diameter 0) (color 0 0 0 0)
-  )
   (junction (at 170.18 120.65) (diameter 0) (color 0 0 0 0)
   )
@@
   (junction (at 124.46 120.65) (diameter 0) (color 0 0 0 0)
   )
+  (junction (at 252.73 90.17) (diameter 0) (color 0 0 0 0)
+  )
   (junction (at 93.98 77.47) (diameter 0) (color 0 0 0 0)
   )
@@
   (junction (at 234.95 154.94) (diameter 0) (color 0 0 0 0)
   )
-  (junction (at 245.11 163.83) (diameter 0) (color 0 0 0 0)
-  )
   (junction (at 154.94 77.47) (diameter 0) (color 0 0 0 0)
   )
@@
   (junction (at 200.66 142.24) (diameter 0) (color 0 0 0 0)
   )
-  (junction (at 260.35 163.83) (diameter 0) (color 0 0 0 0)
-  )
-  (junction (at 229.87 163.83) (diameter 0) (color 0 0 0 0)
-  )
   (junction (at 175.26 133.35) (diameter 0) (color 0 0 0 0)
   )
@@
   (junction (at 80.01 77.47) (diameter 0) (color 0 0 0 0)
   )
-  (junction (at 245.11 120.65) (diameter 0) (color 0 0 0 0)
-  )
   (junction (at 219.71 68.58) (diameter 0) (color 0 0 0 0)
   )
@@
   (junction (at 54.61 154.94) (diameter 0) (color 0 0 0 0)
   )
-  (junction (at 260.35 120.65) (diameter 0) (color 0 0 0 0)
-  )
   (junction (at 229.87 55.88) (diameter 0) (color 0 0 0 0)
   )
@@
   (junction (at 39.37 176.53) (diameter 0) (color 0 0 0 0)
   )
-  (junction (at 260.35 77.47) (diameter 0) (color 0 0 0 0)
-  )
   (junction (at 85.09 68.58) (diameter 0) (color 0 0 0 0)
   )
@@
   (junction (at 190.5 154.94) (diameter 0) (color 0 0 0 0)
   )
-  (junction (at 260.35 142.24) (diameter 0) (color 0 0 0 0)
-  )
   (junction (at 250.19 176.53) (diameter 0) (color 0 0 0 0)
   )
@@
   )
   (no_connect (at 360.68 43.18))
+  (no_connect (at 245.11 142.24))
   (no_connect (at 360.68 71.12))
   (no_connect (at 330.2 43.18))
+  (no_connect (at 260.35 185.42))
+  (no_connect (at 262.89 77.47))
+  (no_connect (at 260.35 142.24))
   (no_connect (at 360.68 68.58))
   (no_connect (at 330.2 45.72))
+  (no_connect (at 245.11 185.42))
+  (no_connect (at 260.35 163.83))
+  (no_connect (at 247.65 77.47))
   (no_connect (at 360.68 63.5))
+  (no_connect (at 245.11 163.83))
+  (no_connect (at 229.87 185.42))
   (no_connect (at 360.68 66.04))
   (wire (pts (xy 229.87 99.06) (xy 229.87 120.65))
@@
     (stroke (width 0) (type default))
   )
-  (wire (pts (xy 260.35 120.65) (xy 260.35 142.24))
-    (stroke (width 0) (type default))
-  )
   (wire (pts (xy 219.71 176.53) (xy 234.95 176.53))
     (stroke (width 0) (type default))
   )
-  (wire (pts (xy 260.35 49.53) (xy 260.35 77.47))
-    (stroke (width 0) (type default))
-  )
   (wire (pts (xy 39.37 176.53) (xy 54.61 176.53))
     (stroke (width 0) (type default))
@@
     (stroke (width 0) (type default))
   )
-  (wire (pts (xy 245.11 142.24) (xy 245.11 163.83))
-    (stroke (width 0) (type default))
-  )
   (wire (pts (xy 34.29 120.65) (xy 34.29 142.24))
     (stroke (width 0) (type default))
@@
     (stroke (width 0) (type default))
   )
-  (wire (pts (xy 229.87 163.83) (xy 229.87 185.42))
-    (stroke (width 0) (type default))
-  )
   (wire (pts (xy 85.09 133.35) (xy 99.06 133.35))
     (stroke (width 0) (type default))
@@
     (stroke (width 0) (type default))
   )
-  (wire (pts (xy 245.11 55.88) (xy 245.11 77.47))
-    (stroke (width 0) (type default))
-  )
   (wire (pts (xy 93.98 163.83) (xy 93.98 185.42))
     (stroke (width 0) (type default))
@@
     (stroke (width 0) (type default))
   )
-  (wire (pts (xy 245.11 163.83) (xy 245.11 185.42))
-    (stroke (width 0) (type default))
-  )
   (wire (pts (xy 367.03 45.72) (xy 360.68 45.72))
     (stroke (width 0) (type default))
@@
     (stroke (width 0) (type default))
   )
-  (wire (pts (xy 245.11 120.65) (xy 245.11 142.24))
-    (stroke (width 0) (type default))
-  )
   (wire (pts (xy 69.85 68.58) (xy 85.09 68.58))
     (stroke (width 0) (type default))
   )
-  (wire (pts (xy 250.19 90.17) (xy 265.43 90.17))
-    (stroke (width 0) (type default))
-  )
   (wire (pts (xy 99.06 176.53) (xy 114.3 176.53))
     (stroke (width 0) (type default))
@@
     (stroke (width 0) (type default))
   )
-  (wire (pts (xy 260.35 77.47) (xy 260.35 99.06))
-    (stroke (width 0) (type default))
-  )
-  (wire (pts (xy 260.35 142.24) (xy 260.35 163.83))
+  (wire (pts (xy 260.35 49.53) (xy 260.35 99.06))
     (stroke (width 0) (type default))
   )
@@
     (stroke (width 0) (type default))
   )
-  (wire (pts (xy 260.35 163.83) (xy 260.35 185.42))
-    (stroke (width 0) (type default))
-  )
   (wire (pts (xy 185.42 120.65) (xy 185.42 142.24))
     (stroke (width 0) (type default))
@@
     (stroke (width 0) (type default))
   )
-  (wire (pts (xy 245.11 77.47) (xy 245.11 99.06))
+  (wire (pts (xy 245.11 55.88) (xy 245.11 99.06))
     (stroke (width 0) (type default))
   )
@@
     (stroke (width 0) (type default))
   )
+  (wire (pts (xy 252.73 90.17) (xy 267.97 90.17))
+    (stroke (width 0) (type default))
+  )
   (wire (pts (xy 205.74 154.94) (xy 219.71 154.94))
     (stroke (width 0) (type default))
@@
     (stroke (width 0) (type default))
   )
-  (wire (pts (xy 234.95 90.17) (xy 250.19 90.17))
+  (wire (pts (xy 234.95 90.17) (xy 252.73 90.17))
     (stroke (width 0) (type default))
   )
@@
     )
   )
-  (symbol (lib_id "ScottoKeebs:Placeholder_Keyswitch") (at 262.89 80.01 0) (unit 1)
+  (symbol (lib_id "ScottoKeebs:Placeholder_Keyswitch") (at 265.43 80.01 0) (unit 1)
     (in_bom yes) (on_board yes) (dnp no) (fields_autoplaced)
-    (property "Reference" "S32" (at 262.89 72.39 0)
+    (property "Reference" "S32" (at 265.43 72.39 0)
       (effects (font (size 1.27 1.27)))
     )
-    (property "Value" "PAD2" (at 262.89 74.93 0)
+    (property "Value" "PAD2" (at 265.43 74.93 0)
       (effects (font (size 1.27 1.27)))
     )
-    (property "Footprint" "ScottoKeebs_MX:MX_PCB_1.00u" (at 262.89 80.01 0)
+    (property "Footprint" "ScottoKeebs_MX:MX_PCB_1.00u" (at 265.43 80.01 0)
       (effects (font (size 1.27 1.27)) hide)
     )
-    (property "Datasheet" "~" (at 262.89 80.01 0)
+    (property "Datasheet" "~" (at 265.43 80.01 0)
       (effects (font (size 1.27 1.27)) hide)
     )
@@
     )
   )
-  (symbol (lib_id "ScottoKeebs:Placeholder_Diode") (at 250.19 86.36 90) (unit 1)
+  (symbol (lib_id "ScottoKeebs:Placeholder_Diode") (at 252.73 86.36 90) (unit 1)
     (in_bom yes) (on_board yes) (dnp no) (fields_autoplaced)
-    (property "Reference" "D31" (at 252.73 85.09 90)
+    (property "Reference" "D31" (at 255.27 85.09 90)
       (effects (font (size 1.27 1.27)) (justify right))
     )
-    (property "Value" "Diode" (at 252.73 87.63 90)
+    (property "Value" "Diode" (at 255.27 87.63 90)
       (effects (font (size 1.27 1.27)) (justify right))
     )
-    (property "Footprint" "ScottoKeebs_Components:Diode_SOD-123" (at 250.19 86.36 0)
+    (property "Footprint" "ScottoKeebs_Components:Diode_SOD-123" (at 252.73 86.36 0)
       (effects (font (size 1.27 1.27)) hide)
     )
-    (property "Datasheet" "" (at 250.19 86.36 0)
+    (property "Datasheet" "" (at 252.73 86.36 0)
       (effects (font (size 1.27 1.27)) hide)
     )
-    (property "Sim.Device" "D" (at 250.19 86.36 0)
+    (property "Sim.Device" "D" (at 252.73 86.36 0)
       (effects (font (size 1.27 1.27)) hide)
     )
-    (property "Sim.Pins" "1=K 2=A" (at 250.19 86.36 0)
+    (property "Sim.Pins" "1=K 2=A" (at 252.73 86.36 0)
       (effects (font (size 1.27 1.27)) hide)
     )
@@
     )
   )
-  (symbol (lib_id "ScottoKeebs:Placeholder_Diode") (at 265.43 86.36 90) (unit 1)
+  (symbol (lib_id "ScottoKeebs:Placeholder_Diode") (at 267.97 86.36 90) (unit 1)
     (in_bom yes) (on_board yes) (dnp no) (fields_autoplaced)
-    (property "Reference" "D32" (at 267.97 85.09 90)
+    (property "Reference" "D32" (at 270.51 85.09 90)
       (effects (font (size 1.27 1.27)) (justify right))
     )
-    (property "Value" "Diode" (at 267.97 87.63 90)
+    (property "Value" "Diode" (at 270.51 87.63 90)
       (effects (font (size 1.27 1.27)) (justify right))
     )
-    (property "Footprint" "ScottoKeebs_Components:Diode_SOD-123" (at 265.43 86.36 0)
+    (property "Footprint" "ScottoKeebs_Components:Diode_SOD-123" (at 267.97 86.36 0)
       (effects (font (size 1.27 1.27)) hide)
     )
-    (property "Datasheet" "" (at 265.43 86.36 0)
+    (property "Datasheet" "" (at 267.97 86.36 0)
       (effects (font (size 1.27 1.27)) hide)
     )
-    (property "Sim.Device" "D" (at 265.43 86.36 0)
+    (property "Sim.Device" "D" (at 267.97 86.36 0)
       (effects (font (size 1.27 1.27)) hide)
     )
-    (property "Sim.Pins" "1=K 2=A" (at 265.43 86.36 0)
+    (property "Sim.Pins" "1=K 2=A" (at 267.97 86.36 0)
       (effects (font (size 1.27 1.27)) hide)
     )
@@
     )
   )
-  (symbol (lib_id "ScottoKeebs:Placeholder_Keyswitch") (at 247.65 80.01 0) (unit 1)
+  (symbol (lib_id "ScottoKeebs:Placeholder_Keyswitch") (at 250.19 80.01 0) (unit 1)
     (in_bom yes) (on_board yes) (dnp no) (fields_autoplaced)
-    (property "Reference" "S31" (at 247.65 72.39 0)
+    (property "Reference" "S31" (at 250.19 72.39 0)
       (effects (font (size 1.27 1.27)))
     )
-    (property "Value" "PAD1" (at 247.65 74.93 0)
+    (property "Value" "PAD1" (at 250.19 74.93 0)
       (effects (font (size 1.27 1.27)))
     )
-    (property "Footprint" "ScottoKeebs_MX:MX_PCB_1.00u" (at 247.65 80.01 0)
+    (property "Footprint" "ScottoKeebs_MX:MX_PCB_1.00u" (at 250.19 80.01 0)
       (effects (font (size 1.27 1.27)) hide)
     )
-    (property "Datasheet" "~" (at 247.65 80.01 0)
+    (property "Datasheet" "~" (at 250.19 80.01 0)
       (effects (font (size 1.27 1.27)) hide)
     )

Commit message: update schema
Parts:
- removed D111, D112, D31, D32, D79, D80, D95, D96: Diode, ScottoKeebs_Components:Diode_SOD-123, symbol ScottoKeebs:Placeholder_Diode
- removed S111: PAD7, ScottoKeebs_MX:MX_PCB_1.00u, symbol ScottoKeebs:Placeholder_Keyswitch
- removed S112: PAD8, ScottoKeebs_MX:MX_PCB_1.00u, symbol ScottoKeebs:Placeholder_Keyswitch
- removed S31: PAD1, ScottoKeebs_MX:MX_PCB_1.00u, symbol ScottoKeebs:Placeholder_Keyswitch
- removed S32: PAD2, ScottoKeebs_MX:MX_PCB_1.00u, symbol ScottoKeebs:Placeholder_Keyswitch
- removed S79: PAD3, ScottoKeebs_MX:MX_PCB_1.00u, symbol ScottoKeebs:Placeholder_Keyswitch
- removed S80: PAD4, ScottoKeebs_MX:MX_PCB_1.00u, symbol ScottoKeebs:Placeholder_Keyswitch
- removed S95: PAD5, ScottoKeebs_MX:MX_PCB_1.00u, symbol ScottoKeebs:Placeholder_Keyswitch
- removed S96: PAD6, ScottoKeebs_MX:MX_PCB_1.00u, symbol ScottoKeebs:Placeholder_Keyswitch
Connections:
- net Col 10: now also S27.1
- net Col 11: now also S28.1; no longer S12.1
- net Col 13: now also S110.1
- net Col 14: now also S12.1
- net Row 0: no longer D12.1 (K)
- net Row 1: now also D12.1 (K)
- no-connect marks 16 -> 7
Other:
- moved on the sheet: D27, D28, S27, S28

Commit message: pcb and schematic v1.0b
Parts:
- added D31: Diode, ScottoKeebs_Components:Diode_SOD-123, symbol ScottoKeebs:Placeholder_Diode
- added D32: BLOC SCORR, LED_THT:LED_D3.0mm, symbol Device:LED
- added D79: CAPS LOCK, LED_THT:LED_D3.0mm, symbol Device:LED
- added D80: BLOC NUM, LED_THT:LED_D3.0mm, symbol Device:LED
- added D95: MIC ON, LED_THT:LED_D3.0mm, symbol Device:LED
- added D96: AUDIO ON, LED_THT:LED_D3.0mm, symbol Device:LED
- added R1, R2, R3, R4, R5: 180, Resistor_THT:R_Axial_DIN0204_L3.6mm_D1.6mm_P7.62mm_Horizontal, symbol ScottoKeebs:Placeholder_Resistor
- added S31: ù, ScottoKeebs_Hotswap:Hotswap_MX_Plated, symbol ScottoKeebs:Placeholder_Keyswitch
- added U2: 4052, Package_SO:TSSOP-16-1EP_4.4x5mm_P0.65mm_EP3x3mm, symbol 4xxx:4052
- S1, S10, S100, S101, S102, S103, S104, S105, S106, S107, S108, S109, S11, S110, S12, S13, S14, S15, S16, S17, S18, S19, S2, S20, S21, S22, S23, S24, S25, S26, S27, S28, S29, S3, S30, S33, S34, S35, S36, S37, S38, S39, S4, S40, S41, S42, S43, S44, S45, S46, S47, S48, S49, S5, S50, S51, S52, S53, S54, S55, S56, S57, S58, S59, S6, S60, S61, S62, S63, S64, S65, S66, S67, S68, S69, S7, S70, S71, S72, S73, S74, S75, S76, S77, S78, S8, S81, S82, S83, S84, S85, S86, S87, S88, S89, S9, S90, S91, S92, S93, S94, S97, S98, S99: footprint ScottoKeebs_MX:MX_PCB_1.00u -> ScottoKeebs_Hotswap:Hotswap_MX_Plated
Connections:
- net +3.3V: now also U2.13 (X), U2.16 (VDD), U2.3 (Y)
- net Col 0: now also U5.23 (I8); no longer S97.1, U5.9 (I0)
- net Col 1: now also U5.22 (I9); no longer S98.1, U5.8 (I1)
- net Col 10: now also S87.1, U5.4 (I5); no longer S107.1, U5.21 (I10)
- net Col 11: now also S12.1, S88.1, U5.5 (I4); no longer S108.1, S92.1, U5.20 (I11)
- net Col 12: now also U5.6 (I3), S31.1; no longer S109.1, S93.1, U5.19 (I12)
- net Col 13: now also S89.1, U5.7 (I2); no longer S110.1, S78.1, S94.1, U5.18 (I13)
- net Col 14: now also S90.1, U5.8 (I1); no longer S12.1, U5.17 (I14)
- net Col 15: now also S16.1, S78.1, U5.9 (I0); no longer U5.16 (I15)
- net Col 2: now also U5.21 (I10); no longer S99.1, U5.7 (I2)
- net Col 3: now also U5.20 (I11); no longer S100.1, U5.6 (I3)
- net Col 4: now also U5.19 (I12); no longer S101.1, S85.1, U5.5 (I4)
- net Col 5: now also U5.18 (I13); no longer S102.1, S86.1, U5.4 (I5)
- net Col 6: now also U5.17 (I14); no longer S103.1, S87.1, U5.3 (I6)
- net Col 7: now also U5.16 (I15); no longer S104.1, S88.1, U5.2 (I7)
- net Col 8: now also S85.1, U5.2 (I7); no longer S105.1, S89.1, U5.23 (I8)
- net Col 9: now also S86.1, U5.3 (I6); no longer S106.1, S90.1, U5.22 (I9)
- net GND: now also D32.1 (K), D79.1 (K), D80.1 (K), D95.1 (K), D96.1 (K), U2.6 (Inh), U2.7 (VEE), U2.8 (VSS)
- net NANO_MUX 1: now also U5.10 (S0); no longer U5.11 (S1)
- net NANO_MUX 2: now also U5.11 (S1); no longer U5.10 (S0)
- net Row 0: now also D100.1 (K), D12.1 (K), D97.1 (K), D98.1 (K), D99.1 (K), U1.11 (D8); no longer U1.5 (D2)
- net Row 1: now also D101.1 (K), D102.1 (K), D103.1 (K), D104.1 (K), U1.10 (D7); no longer D12.1 (K), U1.6 (D3)
- net Row 2: now also D105.1 (K), D106.1 (K), D107.1 (K), U1.9 (D6); no longer U1.7 (D4)
- net Row 3: now also D108.1 (K), D109.1 (K), D110.1 (K)
- net Row 4: now also D92.1 (K), D93.1 (K), D94.1 (K), U1.7 (D4); no longer U1.9 (D6)
- net Row 5: now also U1.6 (D3), D31.1 (K); no longer D85.1 (K), D86.1 (K), D87.1 (K), D88.1 (K), D89.1 (K), D90.1 (K), D92.1 (K), D93.1 (K), D94.1 (K), U1.10 (D7)
- net Row 6: now also D85.1 (K), D86.1 (K), D87.1 (K), D88.1 (K), D89.1 (K), D90.1 (K), U1.5 (D2); no longer D100.1 (K), D101.1 (K), D102.1 (K), D103.1 (K), D104.1 (K), D105.1 (K), D106.1 (K), D107.1 (K), D108.1 (K), D109.1 (K), D110.1 (K), D97.1 (K), D98.1 (K), D99.1 (K), U1.11 (D8)
- net LED_MUX 1: now reaches U1.1 (D1)
- net LED_MUX 1: now also U2.10 (A)
- net Pad Col 0: now reaches U1.13 (D10)
- net Pad Col 0: now also S101.1, S105.1, S108.1, S92.1, S97.1
- net Pad Col 1: now reaches U1.14 (D16)
- net Pad Col 1: now also S102.1, S106.1, S109.1, S98.1
- net Pad Col 2: now reaches U1.15 (D14)
- net Pad Col 2: now also S103.1, S107.1, S110.1, S93.1, S99.1
- net Pad Col 3: now reaches U1.16 (D15)
- net Pad Col 3: now also S100.1, S104.1, S94.1
- net LED_MUX 2: now reaches U1.2 (D0)
- net LED_MUX 2: now also U2.9 (B)
- new net: D79.2 (A), R3.1
- new net: D32.2 (A), R2.1
- new net: D80.2 (A), R1.1
- new net: D96.2 (A), R5.1
- new net: D95.2 (A), R4.1
- new net: D31.2 (A), S31.2
- new net AUDIO ON LED: R5.2, U2.12 (X0)
- new net BLOC NUM LED: R1.2, U2.1 (Y0)
- new net BLOC SCORR LED: R2.2, U2.11 (X3)
- new net CAPS LOCK LED: R3.2, U2.15 (X2)
- new net MIC ON LED: R4.2, U2.14 (X1)
- no-connect marks 7 -> 5
Other:
- company: (none) -> N3 S.r.l. - Andrea Novati
- title: (none) -> K3yb it!
- moved on the sheet: D16, S16, U1, U5

Commit message: added correct footprint soic16
Parts:
- U2: footprint Package_SO:TSSOP-16-1EP_4.4x5mm_P0.65mm_EP3x3mm -> Package_SO:SOP-16_4.55x10.3mm_P1.27mm
Changed lines of the file:
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@@
       (effects (font (size 1.27 1.27)) (justify left))
     )
-    (property "Footprint" "Package_SO:TSSOP-16-1EP_4.4x5mm_P0.65mm_EP3x3mm" (at 179.07 251.46 0)
+    (property "Footprint" "Package_SO:SOP-16_4.55x10.3mm_P1.27mm" (at 179.07 251.46 0)
       (effects (font (size 1.27 1.27)) hide)
     )
