File: k3yb.it/k3yb.it.kicad_sch (KiCad schematic)
At the start: 222 parts, among them SW1 Nice!Nano Reset, U1 Nice_Nano_V2, U2 4052, U5 CD74HC4067M

Commit message: updated footprint added display connector, added battery connector generated new gerber file and drill file major pcb fixes, kostar rotation, mux inverted pinout, key positions
Parts:
- added J1: Display i2c, Connector_JST:JST_GH_SM04B-GHS-TB_1x04-1MP_P1.25mm_Horizontal, symbol Connector:Conn_01x04_Pin
- added J2: Nice Nano i2c, Connector_PinHeader_2.54mm:PinHeader_1x03_P2.54mm_Vertical_SMD_Pin1Left, symbol Connector:Conn_01x03_Pin
- added J3: 18650 battery socket, Connector_JST:JST_PH_S2B-PH-SM4-TB_1x02-1MP_P2.00mm_Horizontal, symbol Connector:Conn_01x02_Pin
Connections:
- net +3.3V: now also U5.1 (COM), J1.3 (Pin_3)
- net GND: now also J1.4 (Pin_4), J3.2 (Pin_2); no longer U5.1 (COM)
- net B+: now reaches U1.24 (B+)
- net B+: now also J3.1 (Pin_1)
- net MIC ON LED renamed LAYER ON LED
- new net SCL: J1.2 (Pin_2), J2.2 (Pin_2)
- new net SDA: J1.1 (Pin_1), J2.1 (Pin_1)
- no-connect marks 1 -> 0
Other:
- added sheet RGB leds (untitled.kicad_sch)

Commit message: updated gerber
Parts:
- J1: footprint Connector_JST:JST_GH_SM04B-GHS-TB_1x04-1MP_P1.25mm_Horizontal -> Connector_JST:JST_PH_B4B-PH-SM4-TB_1x04-1MP_P2.00mm_Vertical
Connections:
- net +3.3V: now also J1.2 (Pin_2); no longer J1.3 (Pin_3)
- net GND: now also J1.1 (Pin_1); no longer J1.4 (Pin_4)
- net SCL: now also J1.3 (Pin_3); no longer J1.2 (Pin_2)
- net SDA: now also J1.4 (Pin_4); no longer J1.1 (Pin_1)
Changed lines of the file:
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@@
 	(wire
 		(pts
-			(xy 54.61 154.94) (xy 69.85 154.94)
+			(xy 292.1 219.71) (xy 290.83 219.71)
 		)
 		(stroke
@@
 	(wire
 		(pts
-			(xy 354.33 77.47) (xy 354.33 97.79)
+			(xy 54.61 154.94) (xy 69.85 154.94)
 		)
 		(stroke
@@
 	(wire
 		(pts
-			(xy 309.88 180.34) (xy 311.15 180.34)
+			(xy 354.33 77.47) (xy 354.33 97.79)
 		)
 		(stroke
@@
 	(wire
 		(pts
-			(xy 309.88 185.42) (xy 321.31 185.42)
+			(xy 309.88 180.34) (xy 321.31 180.34)
 		)
 		(stroke
@@
 	(wire
 		(pts
+			(xy 292.1 217.17) (xy 292.1 219.71)
+		)
+		(stroke
+			(width 0)
+			(type default)
+		)
+	)
+	(wire
+		(pts
 			(xy 34.29 120.65) (xy 34.29 142.24)
 		)
@@
 	(wire
 		(pts
-			(xy 309.88 182.88) (xy 321.31 182.88)
-		)
-		(stroke
-			(width 0)
-			(type default)
-		)
-	)
-	(wire
-		(pts
 			(xy 80.01 142.24) (xy 80.01 163.83)
 		)
@@
 	(wire
 		(pts
-			(xy 309.88 177.8) (xy 311.15 177.8)
+			(xy 309.88 177.8) (xy 325.12 177.8)
 		)
 		(stroke
@@
 	(wire
 		(pts
+			(xy 309.88 185.42) (xy 312.42 185.42)
+		)
+		(stroke
+			(width 0)
+			(type default)
+		)
+	)
+	(wire
+		(pts
 			(xy 160.02 133.35) (xy 175.26 133.35)
 		)
@@
 	(wire
 		(pts
+			(xy 294.64 217.17) (xy 292.1 217.17)
+		)
+		(stroke
+			(width 0)
+			(type default)
+		)
+	)
+	(wire
+		(pts
 			(xy 93.98 77.47) (xy 93.98 99.06)
 		)
@@
 	(wire
 		(pts
+			(xy 309.88 182.88) (xy 312.42 182.88)
+		)
+		(stroke
+			(width 0)
+			(type default)
+		)
+	)
+	(wire
+		(pts
 			(xy 139.7 120.65) (xy 139.7 142.24)
 		)
@@
 	(wire
 		(pts
+			(xy 293.37 204.47) (xy 293.37 200.66)
+		)
+		(stroke
+			(width 0)
+			(type default)
+		)
+	)
+	(wire
+		(pts
 			(xy 214.63 55.88) (xy 214.63 77.47)
 		)
@@
 	(wire
 		(pts
+			(xy 297.18 198.12) (xy 293.37 198.12)
+		)
+		(stroke
+			(width 0)
+			(type default)
+		)
+	)
+	(wire
+		(pts
 			(xy 166.37 240.03) (xy 166.37 241.3)
 		)
@@
 		)
 	)
-	(global_label "SDA"
-		(shape input)
-		(at 311.15 177.8 0)
-		(fields_autoplaced yes)
-		(effects
-			(font
-				(size 1.27 1.27)
-			)
-			(justify left)
-		)
-		(property "Intersheetrefs" "${INTERSHEET_REFS}"
-			(at 317.7033 177.8 0)
-			(effects
-				(font
-					(size 1.27 1.27)
-				)
-				(justify left)
-				(hide yes)
-			)
-		)
-	)
 	(global_label "NANO_MUX 4"
 		(shape output)
@@
 	(global_label "B+"
 		(shape input)
-		(at 293.37 198.12 0)
+		(at 297.18 198.12 0)
+		(fields_autoplaced yes)
+		(effects
+			(font
+				(size 1.27 1.27)
+			)
+			(justify left)
+		)
+		(property "Intersheetrefs" "${INTERSHEET_REFS}"
+			(at 303.0076 198.12 0)
+			(effects
+				(font
+					(size 1.27 1.27)
+				)
+				(justify left)
+				(hide yes)
+			)
+		)
+	)
+	(global_label "SDA"
+		(shape input)
+		(at 312.42 185.42 0)
 		(fields_autoplaced yes)
 		(effects
@@
 		)
 		(property "Intersheetrefs" "${INTERSHEET_REFS}"
-			(at 299.1976 198.12 0)
+			(at 318.9733 185.42 0)
 			(effects
 				(font
@@
 	(global_label "B+"
 		(shape input)
-		(at 290.83 219.71 0)
+		(at 294.64 217.17 0)
 		(fields_autoplaced yes)
 		(effects
@@
 		)
 		(property "Intersheetrefs" "${INTERSHEET_REFS}"
-			(at 296.6576 219.71 0)
+			(at 300.4676 217.17 0)
 			(effects
 				(font
@@
 		)
 	)
-	(global_label "SCL"
+	(global_label "Col 6"
 		(shape input)
-		(at 311.15 180.34 0)
+		(at 124.46 49.53 90)
 		(fields_autoplaced yes)
 		(effects
@@
 		)
 		(property "Intersheetrefs" "${INTERSHEET_REFS}"
-			(at 317.6428 180.34 0)
+			(at 124.46 41.2835 90)
 			(effects
 				(font
@@
 		)
 	)
-	(global_label "Col 6"
+	(global_label "Row 4"
 		(shape input)
-		(at 124.46 49.53 90)
+		(at 260.35 234.95 180)
 		(fields_autoplaced yes)
 		(effects
@@
 				(size 1.27 1.27)
 			)
-			(justify left)
+			(justify right)
 		)
 		(property "Intersheetrefs" "${INTERSHEET_REFS}"
-			(at 124.46 41.2835 90)
+			(at 251.4382 234.95 0)
 			(effects
 				(font
 					(size 1.27 1.27)
 				)
-				(justify left)
+				(justify right)
 				(hide yes)
 			)
 		)
 	)
-	(global_label "Row 4"
+	(global_label "SCL"
 		(shape input)
-		(at 260.35 234.95 180)
+		(at 312.42 182.88 0)
 		(fields_autoplaced yes)
 		(effects
@@
 				(size 1.27 1.27)
 			)
-			(justify right)
+			(justify left)
 		)
 		(property "Intersheetrefs" "${INTERSHEET_REFS}"
-			(at 251.4382 234.95 0)
+			(at 318.9128 182.88 0)
 			(effects
 				(font
 					(size 1.27 1.27)
 				)
-				(justify right)
+				(justify left)
 				(hide yes)
 			)
@@
 	(symbol
 		(lib_id "power:GND")
-		(at 321.31 185.42 0)
+		(at 325.12 177.8 0)
 		(unit 1)
 		(exclude_from_sim no)
@@
 		(fields_autoplaced yes)
 		(property "Reference" "#PWR011"
-			(at 321.31 191.77 0)
+			(at 325.12 184.15 0)
 			(effects
 				(font
@@
 		)
 		(property "Value" "GND"
-			(at 321.31 190.5 0)
+			(at 325.12 182.88 0)
 			(effects
 				(font
@@
 		)
 		(property "Footprint" ""
-			(at 321.31 185.42 0)
+			(at 325.12 177.8 0)
 			(effects
 				(font
@@
 		)
 		(property "Datasheet" ""
-			(at 321.31 185.42 0)
+			(at 325.12 177.8 0)
 			(effects
 				(font
@@
 		)
 		(property "Description" ""
-			(at 321.31 185.42 0)
+			(at 325.12 177.8 0)
 			(effects
 				(font
@@
 			)
 		)
-		(property "Footprint" "Connector_JST:JST_GH_SM04B-GHS-TB_1x04-1MP_P1.25mm_Horizontal"
+		(property "Footprint" "Connector_JST:JST_PH_B4B-PH-SM4-TB_1x04-1MP_P2.00mm_Vertical"
 			(at 304.8 180.34 0)
 			(effects
@@
 	(symbol
 		(lib_id "power:+3.3V")
-		(at 321.31 182.88 0)
+		(at 321.31 180.34 0)
 		(unit 1)
 		(exclude_from_sim no)
@@
 		(dnp no)
 		(property "Reference" "#PWR012"
-			(at 321.31 186.69 0)
+			(at 321.31 184.15 0)
 			(effects
 				(font
@@
 		)
 		(property "Value" "+3.3V"
-			(at 321.31 177.8 0)
+			(at 321.31 175.26 0)
 			(effects
 				(font
@@
 		)
 		(property "Footprint" ""
-			(at 321.31 182.88 0)
+			(at 321.31 180.34 0)
 			(effects
 				(font
@@
 		)
 		(property "Datasheet" ""
-			(at 321.31 182.88 0)
+			(at 321.31 180.34 0)
 			(effects
 				(font
@@
 		)
 		(property "Description" ""
-			(at 321.31 182.88 0)
+			(at 321.31 180.34 0)
 			(effects
 				(font
@@
 	(symbol
 		(lib_id "power:GND")
-		(at 293.37 200.66 0)
+		(at 293.37 204.47 0)
 		(unit 1)
 		(exclude_from_sim no)
@@
 		(fields_autoplaced yes)
 		(property "Reference" "#PWR013"
-			(at 293.37 207.01 0)
+			(at 293.37 210.82 0)
 			(effects
 				(font
@@
 		)
 		(property "Value" "GND"
-			(at 293.37 205.74 0)
+			(at 293.37 209.55 0)
 			(effects
 				(font
@@
 		)
 		(property "Footprint" ""
-			(at 293.37 200.66 0)
+			(at 293.37 204.47 0)
 			(effects
 				(font
@@
 		)
 		(property "Datasheet" ""
-			(at 293.37 200.66 0)
+			(at 293.37 204.47 0)
 			(effects
 				(font
@@
 		)
 		(property "Description" ""
-			(at 293.37 200.66 0)
+			(at 293.37 204.47 0)
 			(effects
 				(font
